Commit message: dimension change

File: src/diff_drive_robot-main/urdf/robot_core.xacro (robot description, xacro)
@@ -2,7 +2,5 @@
 <robot name="car_robot" xmlns:xacro="http://www.ros.org/wiki/xacro" xmlns:gazebo="http://gazebo.apache.org/xmlns/gazebo">
   <xacro:include filename="inertial_macros.xacro" />
-  <!-- Base Link -->
   <link name="base_link"/>
-  <!-- Chassis -->
   <joint name="chassis_joint" type="fixed">
     <parent link="base_link"/>
@@ -12,7 +10,7 @@
   <link name="chassis">
     <visual>
-      <origin xyz="0.15 0 0.075"/>
+      <origin xyz="0.25 0 0.075"/>
       <geometry>
-        <box size="0.3 0.3 0.15"/>
+        <box size="0.5 0.3 0.15"/>
       </geometry>
       <material name="chassis_material">
@@ -21,7 +19,7 @@
     </visual>
     <collision>
-      <origin xyz="0.15 0 0.075"/>
+      <origin xyz="0.25 0 0.075"/>
       <geometry>
-        <box size="0.3 0.3 0.15"/>
+        <box size="0.5 0.3 0.15"/>
       </geometry>
     </collision>
@@ -34,5 +32,5 @@
     <parent link="base_link"/>
     <child link="left_wheel"/>
-    <origin xyz="0 0.175 0" rpy="-1.57 0 0"/>
+    <origin xyz="0.1 0.175 0" rpy="-1.57 0 0"/>
     <axis xyz="0 0 1"/>
   </joint>
@@ -40,5 +38,5 @@
     <visual>
       <geometry>
-        <cylinder radius="0.05" length="0.04"/>
+        <cylinder radius="0.075" length="0.04"/>
       </geometry>
       <material name="wheel_material">
@@ -48,8 +46,8 @@
     <collision>
       <geometry>
-        <cylinder radius="0.05" length="0.04"/>
+        <cylinder radius="0.075" length="0.04"/>
       </geometry>
     </collision>
-        <xacro:inertial_cylinder mass="0.1" length="0.04" radius="0.05">
+        <xacro:inertial_cylinder mass="0.1" length="0.04" radius="0.075">
             <origin xyz="0 0 0" rpy="0 0 0"/>
          </xacro:inertial_cylinder>
@@ -58,5 +56,5 @@
     <parent link="base_link"/>
     <child link="right_wheel"/>
-    <origin xyz="0 -0.175 0" rpy="1.57 0 0"/>
+    <origin xyz="0.1 -0.175 0" rpy="1.57 0 0"/>
     <axis xyz="0 0 -1"/>
   </joint>
@@ -64,5 +62,5 @@
     <visual>
       <geometry>
-        <cylinder radius="0.05" length="0.04"/>
+        <cylinder radius="0.075" length="0.04"/>
       </geometry>
       <material name="wheel_material">
@@ -72,8 +70,8 @@
     <collision>
       <geometry>
-        <cylinder radius="0.05" length="0.04"/>
+        <cylinder radius="0.075" length="0.04"/>
       </geometry>
     </collision>
-        <xacro:inertial_cylinder mass="0.1" length="0.04" radius="0.05">
+        <xacro:inertial_cylinder mass="0.1" length="0.04" radius="0.075">
             <origin xyz="0 0 0" rpy="0 0 0"/>
          </xacro:inertial_cylinder>
@@ -83,5 +81,5 @@
     <parent link="base_link"/>
     <child link="left_front_wheel"/>
-    <origin xyz="0.14 0.175 0" rpy="-1.57 0 0"/>
+    <origin xyz="0.4 0.175 0" rpy="-1.57 0 0"/>
     <axis xyz="0 0 1"/>
   </joint>
@@ -89,5 +87,5 @@
     <visual>
       <geometry>
-        <cylinder radius="0.05" length="0.04"/>
+        <cylinder radius="0.075" length="0.04"/>
       </geometry>
       <material name="wheel_material">
@@ -97,8 +95,8 @@
     <collision>
       <geometry>
-        <cylinder radius="0.05" length="0.04"/>
+        <cylinder radius="0.075" length="0.04"/>
       </geometry>
     </collision>
-        <xacro:inertial_cylinder mass="0.1" length="0.04" radius="0.05">
+        <xacro:inertial_cylinder mass="0.1" length="0.04" radius="0.075">
             <origin xyz="0 0 0" rpy="0 0 0"/>
          </xacro:inertial_cylinder>
@@ -107,5 +105,5 @@
     <parent link="base_link"/>
     <child link="right_front_wheel"/>
-    <origin xyz="0.14 -0.175 0" rpy="1.57 0 0"/>
+    <origin xyz="0.4 -0.175 0" rpy="1.57 0 0"/>
     <axis xyz="0 0 -1"/>
   </joint>
@@ -113,5 +111,5 @@
     <visual>
       <geometry>
-        <cylinder radius="0.05" length="0.04"/>
+        <cylinder radius="0.075" length="0.04"/>
       </geometry>
       <material name="wheel_material">
@@ -121,8 +119,8 @@
     <collision>
       <geometry>
-        <cylinder radius="0.05" length="0.04"/>
+        <cylinder radius="0.075" length="0.04"/>
       </geometry>
     </collision>
-        <xacro:inertial_cylinder mass="0.1" length="0.04" radius="0.05">
+        <xacro:inertial_cylinder mass="0.1" length="0.04" radius="0.075">
             <origin xyz="0 0 0" rpy="0 0 0"/>
          </xacro:inertial_cylinder>

Commit message: minor change

File: src/diff_drive_robot-main/urdf/robot_core.xacro (robot description, xacro)
@@ -2,5 +2,7 @@
 <robot name="car_robot" xmlns:xacro="http://www.ros.org/wiki/xacro" xmlns:gazebo="http://gazebo.apache.org/xmlns/gazebo">
   <xacro:include filename="inertial_macros.xacro" />
+  <!-- Base Link -->
   <link name="base_link"/>
+  <!-- Chassis -->
   <joint name="chassis_joint" type="fixed">
     <parent link="base_link"/>
@@ -10,7 +12,7 @@
   <link name="chassis">
     <visual>
-      <origin xyz="0.25 0 0.075"/>
+      <origin xyz="0.275 0 0.075"/>
       <geometry>
-        <box size="0.5 0.3 0.15"/>
+        <box size="0.55 0.4 0.15"/>
       </geometry>
       <material name="chassis_material">
@@ -19,11 +21,11 @@
     </visual>
     <collision>
-      <origin xyz="0.25 0 0.075"/>
+      <origin xyz="0.275 0 0.075"/>
       <geometry>
-        <box size="0.5 0.3 0.15"/>
+        <box size="0.55 0.34 0.15"/>
       </geometry>
     </collision>
-      <xacro:inertial_box mass="0.5" x="0.3" y="0.3" z="0.15">
-            <origin xyz="0.15 0 0.075" rpy="0 0 0"/>
+      <xacro:inertial_box mass="0.5" x="0.55" y="0.4" z="0.15">
+            <origin xyz="0.275 0 0.075" rpy="0 0 0"/>
          </xacro:inertial_box>
   </link>
@@ -32,5 +34,5 @@
     <parent link="base_link"/>
     <child link="left_wheel"/>
-    <origin xyz="0.1 0.175 0" rpy="-1.57 0 0"/>
+    <origin xyz="-0.1 0.225 0" rpy="-1.57 0 0"/>
     <axis xyz="0 0 1"/>
   </joint>
@@ -56,5 +58,5 @@
     <parent link="base_link"/>
     <child link="right_wheel"/>
-    <origin xyz="0.1 -0.175 0" rpy="1.57 0 0"/>
+    <origin xyz="-0.1 -0.225 0" rpy="1.57 0 0"/>
     <axis xyz="0 0 -1"/>
   </joint>
@@ -81,5 +83,5 @@
     <parent link="base_link"/>
     <child link="left_front_wheel"/>
-    <origin xyz="0.4 0.175 0" rpy="-1.57 0 0"/>
+    <origin xyz="0.3 0.225 0" rpy="-1.57 0 0"/>
     <axis xyz="0 0 1"/>
   </joint>
@@ -105,5 +107,5 @@
     <parent link="base_link"/>
     <child link="right_front_wheel"/>
-    <origin xyz="0.4 -0.175 0" rpy="1.57 0 0"/>
+    <origin xyz="0.3 -0.225 0" rpy="1.57 0 0"/>
     <axis xyz="0 0 -1"/>
   </joint>

Commit message: minor change

File: src/diff_drive_robot-main/urdf/robot_core.xacro (robot description, xacro)
@@ -34,5 +34,5 @@
     <parent link="base_link"/>
     <child link="left_wheel"/>
-    <origin xyz="-0.1 0.225 0" rpy="-1.57 0 0"/>
+    <origin xyz="0 0.225 0" rpy="-1.57 0 0"/>
     <axis xyz="0 0 1"/>
   </joint>
@@ -58,5 +58,5 @@
     <parent link="base_link"/>
     <child link="right_wheel"/>
-    <origin xyz="-0.1 -0.225 0" rpy="1.57 0 0"/>
+    <origin xyz="0 -0.225 0" rpy="1.57 0 0"/>
     <axis xyz="0 0 -1"/>
   </joint>

Commit message: added basefootprint

File: src/diff_drive_robot-main/urdf/robot_core.xacro (robot description, xacro)
@@ -4,4 +4,24 @@
   <!-- Base Link -->
   <link name="base_link"/>
+  <link name="base_footprint">
+    <collision>
+      <geometry>
+        <box size="0.55 0.4 0.01"/>
+      </geometry>
+    </collision>
+    <visual>
+      <geometry>
+        <box size="0.55 0.4 0.01"/>
+      </geometry>
+      <material name="footprint_material">
+        <color rgba="0.0 0.0 1.0 0.5"/>
+      </material>
+    </visual>
+  </link>
+  <joint name="base_footprint_joint" type="fixed">
+    <parent link="base_link"/>
+    <child link="base_footprint"/>
+    <origin xyz="0 0 -0.05"/>
+  </joint>
   <!-- Chassis -->
   <joint name="chassis_joint" type="fixed">
