Commit message: fix multirobot tf

File: src/diff_drive_robot-main/urdf/gazebo_control.xacro (robot description, xacro)
@@ -1,4 +1,7 @@
 <?xml version="1.0"?>
 <robot xmlns:xacro="http://www.ros.org/wiki/xacro">
+  <!-- namespace arg: pass the robot namespace so TF frame IDs are unique per robot -->
+  <xacro:arg name="namespace" default=""/>
+  <xacro:property name="ns" value="$(arg namespace)"/>
    <gazebo>
       <plugin filename="libgz-sim-diff-drive-system" name="gz::sim::systems::DiffDrive">
@@ -14,8 +17,9 @@
     <max_linear_speed>2.0</max_linear_speed>
     <max_angular_speed>3.14</max_angular_speed>
-            <odom_topic>odom</odom_topic>
-         <frame_id>odom</frame_id>
-         <child_frame_id>base_link</child_frame_id>
-             <tf_topic>/tf</tf_topic>
+    <odom_topic>odom</odom_topic>
+    <!-- frame IDs include namespace prefix so they are unique across robots -->
+    <frame_id>${ns + '/odom' if ns else 'odom'}</frame_id>
+    <child_frame_id>${ns + '/base_link' if ns else 'base_link'}</child_frame_id>
+    <tf_topic>/tf</tf_topic>
     <!-- Add debug topics -->
     <debug>true</debug>
