Commit message: Namespace Gazebo sensor topics

File: src/diff_drive_robot-main/urdf/camera.xacro (robot description, xacro)
@@ -1,4 +1,6 @@
 <?xml version="1.0"?>
 <robot xmlns:xacro="http://www.ros.org/wiki/xacro">
+  <xacro:arg name="namespace" default=""/>
+  <xacro:property name="ns" value="$(arg namespace)"/>
   <!-- RGB camera: front-top of chassis, 60° FOV, 640x480 @ 30 Hz -->
   <joint name="camera_joint" type="fixed">
@@ -32,6 +34,6 @@
       <always_on>true</always_on>
       <update_rate>30</update_rate>
-      <topic>/camera/image_raw</topic>
-      <gz_frame_id>camera_optical_frame</gz_frame_id>
+      <topic>${ns + '/camera/image_raw' if ns else 'camera/image_raw'}</topic>
+      <gz_frame_id>${ns + '/camera_optical_frame' if ns else 'camera_optical_frame'}</gz_frame_id>
       <camera>
         <horizontal_fov>1.047</horizontal_fov>

File: src/diff_drive_robot-main/urdf/gazebo_control.xacro (robot description, xacro)
@@ -11,5 +11,5 @@
     <wheel_radius>0.1</wheel_radius>
     <odom_publish_frequency>50</odom_publish_frequency>
-    <topic>cmd_vel</topic>
+    <topic>${ns + '/cmd_vel' if ns else 'cmd_vel'}</topic>
     <!-- PID controllers -->
     <wheel_acceleration>1.0</wheel_acceleration>
@@ -17,5 +17,5 @@
     <max_linear_speed>2.0</max_linear_speed>
     <max_angular_speed>3.14</max_angular_speed>
-    <odom_topic>odom</odom_topic>
+    <odom_topic>${ns + '/odom' if ns else 'odom'}</odom_topic>
     <!-- frame IDs include namespace prefix so they are unique across robots -->
     <frame_id>${ns + '/odom' if ns else 'odom'}</frame_id>

File: src/diff_drive_robot-main/urdf/lidar.xacro (robot description, xacro)
@@ -1,4 +1,6 @@
 <?xml version="1.0"?>
 <robot xmlns:xacro="http://www.ros.org/wiki/xacro" >
+   <xacro:arg name="namespace" default=""/>
+   <xacro:property name="ns" value="$(arg namespace)"/>
    <joint name="laser_joint" type="fixed">
      <parent link="chassis"/>
@@ -33,6 +35,6 @@
          <visualize>true</visualize>
          <update_rate>10</update_rate>
-         <topic>scan</topic>
-         <gz_frame_id>laser_frame</gz_frame_id>
+         <topic>${ns + '/scan' if ns else 'scan'}</topic>
+         <gz_frame_id>${ns + '/laser_frame' if ns else 'laser_frame'}</gz_frame_id>
          <lidar>
             <scan>

File: src/diff_drive_robot-main/urdf/lidar3d.xacro (robot description, xacro)
@@ -11,4 +11,6 @@
 -->
 <robot xmlns:xacro="http://www.ros.org/wiki/xacro">
+  <xacro:arg name="namespace" default=""/>
+  <xacro:property name="ns" value="$(arg namespace)"/>
   <!-- Mount at same position as 2D lidar so Nav2 costmaps still work -->
   <joint name="laser_joint" type="fixed">
@@ -44,6 +46,6 @@
       <visualize>false</visualize>
       <update_rate>10</update_rate>
-      <topic>points</topic>
-      <gz_frame_id>laser_frame</gz_frame_id>
+      <topic>${ns + '/points' if ns else 'points'}</topic>
+      <gz_frame_id>${ns + '/laser_frame' if ns else 'laser_frame'}</gz_frame_id>
       <lidar>
         <scan>
