Commit message: Tune sim performance, add camera toggle

File: src/rosnav_bot/urdf/lidar.xacro (robot description, xacro)
@@ -6,5 +6,5 @@
      <parent link="chassis"/>
      <child link="laser_frame"/>
-     <origin xyz="0.1 0 0.175" rpy="0 0 0"/>
+     <origin xyz="0.45 0 0.175" rpy="0 0 0"/>
    </joint>
    <link name="laser_frame">

File: src/rosnav_bot/urdf/robot.urdf.xacro (robot description, xacro)
@@ -10,4 +10,7 @@
         <xacro:include filename="lidar.xacro" />
     </xacro:unless>
-    <xacro:include filename="camera.xacro" />
+    <xacro:arg name="enable_camera" default="false"/>
+    <xacro:if value="${'$(arg enable_camera)' == 'true'}">
+        <xacro:include filename="camera.xacro" />
+    </xacro:if>
 </robot>
