Commit message: tune SLAM and EKF configs

File: src/rosnav_bot/urdf/robot_core.xacro (robot description, xacro)
@@ -68,5 +68,5 @@
     <collision>
       <geometry>
-        <cylinder radius="0.075" length="0.04"/>
+        <sphere radius="0.075"/>
       </geometry>
     </collision>
@@ -92,5 +92,5 @@
     <collision>
       <geometry>
-        <cylinder radius="0.075" length="0.04"/>
+        <sphere radius="0.075"/>
       </geometry>
     </collision>
@@ -117,5 +117,5 @@
     <collision>
       <geometry>
-        <cylinder radius="0.075" length="0.04"/>
+        <sphere radius="0.075"/>
       </geometry>
     </collision>
@@ -141,5 +141,5 @@
     <collision>
       <geometry>
-        <cylinder radius="0.075" length="0.04"/>
+        <sphere radius="0.075"/>
       </geometry>
     </collision>

Commit message: add bench scripts, fusion updates

File: src/rosnav_bot/urdf/robot_core.xacro (robot description, xacro)
@@ -10,12 +10,4 @@
       </geometry>
     </collision>
-    <visual>
-      <geometry>
-        <box size="0.55 0.4 0.01"/>
-      </geometry>
-      <material name="footprint_material">
-        <color rgba="0.0 0.0 1.0 0.5"/>
-      </material>
-    </visual>
   </link>
   <joint name="base_footprint_joint" type="fixed">
@@ -31,12 +23,39 @@
   </joint>
   <link name="chassis">
-    <visual>
-      <origin xyz="0.275 0 0.075"/>
-      <geometry>
-        <box size="0.55 0.4 0.15"/>
-      </geometry>
-      <material name="chassis_material">
-        <color rgba="0.40 0.23 0.72 1.0"/>
-      </material>
+    <!-- Lower skirt -->
+    <visual>
+      <origin xyz="0.275 0 0.05"/>
+      <geometry><box size="0.55 0.40 0.10"/></geometry>
+      <material name="skirt_material"><color rgba="0.16 0.16 0.18 1.0"/></material>
+    </visual>
+    <!-- Upper shell -->
+    <visual>
+      <origin xyz="0.275 0 0.125"/>
+      <geometry><box size="0.53 0.38 0.05"/></geometry>
+      <material name="chassis_material"><color rgba="0.40 0.23 0.72 1.0"/></material>
+    </visual>
+    <!-- Top accent plate -->
+    <visual>
+      <origin xyz="0.25 0 0.151"/>
+      <geometry><box size="0.40 0.30 0.004"/></geometry>
+      <material name="accent_material"><color rgba="0.62 0.50 0.88 1.0"/></material>
+    </visual>
+    <!-- Front bumper -->
+    <visual>
+      <origin xyz="0.56 0 0.04"/>
+      <geometry><box size="0.02 0.40 0.05"/></geometry>
+      <material name="bumper_material"><color rgba="0.08 0.08 0.09 1.0"/></material>
+    </visual>
+    <!-- Front status LED strip -->
+    <visual>
+      <origin xyz="0.541 0 0.125"/>
+      <geometry><box size="0.004 0.30 0.012"/></geometry>
+      <material name="led_material"><color rgba="0.1 0.9 1.0 1.0"/></material>
+    </visual>
+    <!-- Lidar mount ring -->
+    <visual>
+      <origin xyz="0.45 0 0.1555"/>
+      <geometry><cylinder radius="0.06" length="0.01"/></geometry>
+      <material name="bumper_material"><color rgba="0.08 0.08 0.09 1.0"/></material>
     </visual>
     <collision>
@@ -63,6 +82,10 @@
       </geometry>
       <material name="wheel_material">
-        <color rgba="0 0 0 1.0"/>
-      </material>
+        <color rgba="0.05 0.05 0.05 1.0"/>
+      </material>
+    </visual>
+    <visual>
+      <geometry><cylinder radius="0.045" length="0.044"/></geometry>
+      <material name="hub_material"><color rgba="0.70 0.70 0.74 1.0"/></material>
     </visual>
     <collision>
@@ -87,6 +110,10 @@
       </geometry>
       <material name="wheel_material">
-        <color rgba="0 0 0 1.0"/>
-      </material>
+        <color rgba="0.05 0.05 0.05 1.0"/>
+      </material>
+    </visual>
+    <visual>
+      <geometry><cylinder radius="0.045" length="0.044"/></geometry>
+      <material name="hub_material"><color rgba="0.70 0.70 0.74 1.0"/></material>
     </visual>
     <collision>
@@ -112,6 +139,10 @@
       </geometry>
       <material name="wheel_material">
-        <color rgba="0 0 0 1.0"/>
-      </material>
+        <color rgba="0.05 0.05 0.05 1.0"/>
+      </material>
+    </visual>
+    <visual>
+      <geometry><cylinder radius="0.045" length="0.044"/></geometry>
+      <material name="hub_material"><color rgba="0.70 0.70 0.74 1.0"/></material>
     </visual>
     <collision>
@@ -136,6 +167,10 @@
       </geometry>
       <material name="wheel_material">
-        <color rgba="0 0 0 1.0"/>
-      </material>
+        <color rgba="0.05 0.05 0.05 1.0"/>
+      </material>
+    </visual>
+    <visual>
+      <geometry><cylinder radius="0.045" length="0.044"/></geometry>
+      <material name="hub_material"><color rgba="0.70 0.70 0.74 1.0"/></material>
     </visual>
     <collision>

File: src/rosnav_bot/urdf/robot_core_ackermann.xacro (robot description, xacro)
@@ -10,12 +10,4 @@
       </geometry>
     </collision>
-    <visual>
-      <geometry>
-        <box size="0.65 0.4 0.01"/>
-      </geometry>
-      <material name="footprint_material">
-        <color rgba="0.0 0.0 1.0 0.5"/>
-      </material>
-    </visual>
   </link>
   <joint name="base_footprint_joint" type="fixed">
@@ -32,11 +24,27 @@
   <link name="chassis">
     <visual>
-      <origin xyz="0.3 0 0.075"/>
-      <geometry>
-        <box size="0.65 0.35 0.15"/>
-      </geometry>
-      <material name="chassis_material">
-        <color rgba="0.72 0.23 0.10 1.0"/>
-      </material>
+      <origin xyz="0.3 0 0.05"/>
+      <geometry><box size="0.65 0.35 0.10"/></geometry>
+      <material name="skirt_material"><color rgba="0.16 0.16 0.18 1.0"/></material>
+    </visual>
+    <visual>
+      <origin xyz="0.3 0 0.125"/>
+      <geometry><box size="0.63 0.33 0.05"/></geometry>
+      <material name="chassis_material"><color rgba="0.72 0.23 0.10 1.0"/></material>
+    </visual>
+    <visual>
+      <origin xyz="0.27499999999999997 0 0.151"/>
+      <geometry><box size="0.50 0.25 0.004"/></geometry>
+      <material name="accent_material"><color rgba="0.62 0.50 0.88 1.0"/></material>
+    </visual>
+    <visual>
+      <origin xyz="0.635 0 0.04"/>
+      <geometry><box size="0.02 0.35 0.05"/></geometry>
+      <material name="bumper_material"><color rgba="0.08 0.08 0.09 1.0"/></material>
+    </visual>
+    <visual>
+      <origin xyz="0.616 0 0.125"/>
+      <geometry><box size="0.004 0.25 0.012"/></geometry>
+      <material name="led_material"><color rgba="0.1 0.9 1.0 1.0"/></material>
     </visual>
     <collision>
@@ -63,6 +71,10 @@
       </geometry>
       <material name="wheel_material">
-        <color rgba="0 0 0 1.0"/>
-      </material>
+        <color rgba="0.05 0.05 0.05 1.0"/>
+      </material>
+    </visual>
+    <visual>
+      <geometry><cylinder radius="0.045" length="0.044"/></geometry>
+      <material name="hub_material"><color rgba="0.70 0.70 0.74 1.0"/></material>
     </visual>
     <collision>
@@ -87,6 +99,10 @@
       </geometry>
       <material name="wheel_material">
-        <color rgba="0 0 0 1.0"/>
-      </material>
+        <color rgba="0.05 0.05 0.05 1.0"/>
+      </material>
+    </visual>
+    <visual>
+      <geometry><cylinder radius="0.045" length="0.044"/></geometry>
+      <material name="hub_material"><color rgba="0.70 0.70 0.74 1.0"/></material>
     </visual>
     <collision>
@@ -139,6 +155,10 @@
       </geometry>
       <material name="wheel_material">
-        <color rgba="0 0 0 1.0"/>
-      </material>
+        <color rgba="0.05 0.05 0.05 1.0"/>
+      </material>
+    </visual>
+    <visual>
+      <geometry><cylinder radius="0.045" length="0.044"/></geometry>
+      <material name="hub_material"><color rgba="0.70 0.70 0.74 1.0"/></material>
     </visual>
     <collision>
@@ -188,6 +208,10 @@
       </geometry>
       <material name="wheel_material">
-        <color rgba="0 0 0 1.0"/>
-      </material>
+        <color rgba="0.05 0.05 0.05 1.0"/>
+      </material>
+    </visual>
+    <visual>
+      <geometry><cylinder radius="0.045" length="0.044"/></geometry>
+      <material name="hub_material"><color rgba="0.70 0.70 0.74 1.0"/></material>
     </visual>
     <collision>

File: src/rosnav_bot/urdf/robot_core_mecanum.xacro (robot description, xacro)
@@ -10,12 +10,4 @@
       </geometry>
     </collision>
-    <visual>
-      <geometry>
-        <box size="0.55 0.4 0.01"/>
-      </geometry>
-      <material name="footprint_material">
-        <color rgba="0.0 0.0 1.0 0.5"/>
-      </material>
-    </visual>
   </link>
   <joint name="base_footprint_joint" type="fixed">
@@ -32,11 +24,27 @@
   <link name="chassis">
     <visual>
-      <origin xyz="0.275 0 0.075"/>
-      <geometry>
-        <box size="0.55 0.4 0.15"/>
-      </geometry>
-      <material name="chassis_material">
-        <color rgba="0.40 0.23 0.72 1.0"/>
-      </material>
+      <origin xyz="0.275 0 0.05"/>
+      <geometry><box size="0.55 0.4 0.10"/></geometry>
+      <material name="skirt_material"><color rgba="0.16 0.16 0.18 1.0"/></material>
+    </visual>
+    <visual>
+      <origin xyz="0.275 0 0.125"/>
+      <geometry><box size="0.53 0.38 0.05"/></geometry>
+      <material name="chassis_material"><color rgba="0.40 0.23 0.72 1.0"/></material>
+    </visual>
+    <visual>
+      <origin xyz="0.25 0 0.151"/>
+      <geometry><box size="0.40 0.30 0.004"/></geometry>
+      <material name="accent_material"><color rgba="0.62 0.50 0.88 1.0"/></material>
+    </visual>
+    <visual>
+      <origin xyz="0.56 0 0.04"/>
+      <geometry><box size="0.02 0.4 0.05"/></geometry>
+      <material name="bumper_material"><color rgba="0.08 0.08 0.09 1.0"/></material>
+    </visual>
+    <visual>
+      <origin xyz="0.541 0 0.125"/>
+      <geometry><box size="0.004 0.30 0.012"/></geometry>
+      <material name="led_material"><color rgba="0.1 0.9 1.0 1.0"/></material>
     </visual>
     <collision>
@@ -63,6 +71,10 @@
       </geometry>
       <material name="wheel_material">
-        <color rgba="0 0 0 1.0"/>
+        <color rgba="0.05 0.05 0.05 1.0"/>
       </material>
+    </visual>
+    <visual>
+      <geometry><cylinder radius="0.045" length="0.044"/></geometry>
+      <material name="hub_material"><color rgba="0.70 0.70 0.74 1.0"/></material>
     </visual>
     <collision>
@@ -87,6 +99,10 @@
       </geometry>
       <material name="wheel_material">
-        <color rgba="0 0 0 1.0"/>
+        <color rgba="0.05 0.05 0.05 1.0"/>
       </material>
+    </visual>
+    <visual>
+      <geometry><cylinder radius="0.045" length="0.044"/></geometry>
+      <material name="hub_material"><color rgba="0.70 0.70 0.74 1.0"/></material>
     </visual>
     <collision>
@@ -112,6 +128,10 @@
       </geometry>
       <material name="wheel_material">
-        <color rgba="0 0 0 1.0"/>
+        <color rgba="0.05 0.05 0.05 1.0"/>
       </material>
+    </visual>
+    <visual>
+      <geometry><cylinder radius="0.045" length="0.044"/></geometry>
+      <material name="hub_material"><color rgba="0.70 0.70 0.74 1.0"/></material>
     </visual>
     <collision>
@@ -136,6 +156,10 @@
       </geometry>
       <material name="wheel_material">
-        <color rgba="0 0 0 1.0"/>
+        <color rgba="0.05 0.05 0.05 1.0"/>
       </material>
+    </visual>
+    <visual>
+      <geometry><cylinder radius="0.045" length="0.044"/></geometry>
+      <material name="hub_material"><color rgba="0.70 0.70 0.74 1.0"/></material>
     </visual>
     <collision>

File: src/rosnav_bot/urdf/robot_core_outdoor.xacro (robot description, xacro)
@@ -8,12 +8,4 @@
   <link name="base_link"/>
   <link name="base_footprint">
-    <visual>
-      <geometry>
-        <box size="0.55 0.4 0.01"/>
-      </geometry>
-      <material name="footprint_material">
-        <color rgba="0.0 0.0 1.0 0.5"/>
-      </material>
-    </visual>
   </link>
   <joint name="base_footprint_joint" type="fixed">
@@ -30,11 +22,27 @@
   <link name="chassis">
     <visual>
-      <origin xyz="0.275 0 0.075"/>
-      <geometry>
-        <box size="0.55 0.4 0.15"/>
-      </geometry>
-      <material name="chassis_material">
-        <color rgba="0.40 0.23 0.72 1.0"/>
-      </material>
+      <origin xyz="0.275 0 0.05"/>
+      <geometry><box size="0.55 0.4 0.10"/></geometry>
+      <material name="skirt_material"><color rgba="0.16 0.16 0.18 1.0"/></material>
+    </visual>
+    <visual>
+      <origin xyz="0.275 0 0.125"/>
+      <geometry><box size="0.53 0.38 0.05"/></geometry>
+      <material name="chassis_material"><color rgba="0.40 0.23 0.72 1.0"/></material>
+    </visual>
+    <visual>
+      <origin xyz="0.25 0 0.151"/>
+      <geometry><box size="0.40 0.30 0.004"/></geometry>
+      <material name="accent_material"><color rgba="0.62 0.50 0.88 1.0"/></material>
+    </visual>
+    <visual>
+      <origin xyz="0.56 0 0.04"/>
+      <geometry><box size="0.02 0.4 0.05"/></geometry>
+      <material name="bumper_material"><color rgba="0.08 0.08 0.09 1.0"/></material>
+    </visual>
+    <visual>
+      <origin xyz="0.541 0 0.125"/>
+      <geometry><box size="0.004 0.30 0.012"/></geometry>
+      <material name="led_material"><color rgba="0.1 0.9 1.0 1.0"/></material>
     </visual>
     <collision>
@@ -61,6 +69,10 @@
       </geometry>
       <material name="wheel_material">
-        <color rgba="0 0 0 1.0"/>
+        <color rgba="0.05 0.05 0.05 1.0"/>
       </material>
+    </visual>
+    <visual>
+      <geometry><cylinder radius="0.096" length="0.054"/></geometry>
+      <material name="hub_material"><color rgba="0.70 0.70 0.74 1.0"/></material>
     </visual>
     <collision>
@@ -85,6 +97,10 @@
       </geometry>
       <material name="wheel_material">
-        <color rgba="0 0 0 1.0"/>
+        <color rgba="0.05 0.05 0.05 1.0"/>
       </material>
+    </visual>
+    <visual>
+      <geometry><cylinder radius="0.096" length="0.054"/></geometry>
+      <material name="hub_material"><color rgba="0.70 0.70 0.74 1.0"/></material>
     </visual>
     <collision>
@@ -110,6 +126,10 @@
       </geometry>
       <material name="wheel_material">
-        <color rgba="0 0 0 1.0"/>
+        <color rgba="0.05 0.05 0.05 1.0"/>
       </material>
+    </visual>
+    <visual>
+      <geometry><cylinder radius="0.096" length="0.054"/></geometry>
+      <material name="hub_material"><color rgba="0.70 0.70 0.74 1.0"/></material>
     </visual>
     <collision>
@@ -134,6 +154,10 @@
       </geometry>
       <material name="wheel_material">
-        <color rgba="0 0 0 1.0"/>
+        <color rgba="0.05 0.05 0.05 1.0"/>
       </material>
+    </visual>
+    <visual>
+      <geometry><cylinder radius="0.096" length="0.054"/></geometry>
+      <material name="hub_material"><color rgba="0.70 0.70 0.74 1.0"/></material>
     </visual>
     <collision>
